File: telegram control.kicad_sch (KiCad schematic)
At the start: 13 parts, among them J1 Screw_Terminal_01x03, J2 Screw_Terminal_01x02, K1 SANYOU_SRD_Form_C, Q1 MMBT3904, U1 ESP32-C3_SUPERMINI_TH, U3 L7805

Commit message: telegram_control
Connections:
- net +5V: now also C2.1, U3.3 (OUT)
Changed lines of the file:
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@@
 	(paper "A4")
+	(junction
+		(at 210.82 31.75)
+		(diameter 0)
+		(color 0 0 0 0)
+	)
 	(junction
 		(at 232.41 53.34)
@@
 					(unit 1)
 				)
+			)
+		)
+	)
+	(symbol
+		(lib_id "power:+5V")
+		(at 210.82 31.75 0)
+		(unit 1)
+		(exclude_from_sim no)
+		(in_bom yes)
+		(on_board yes)
+		(dnp no)
+		(fields_autoplaced yes)
+		(property "Reference" "#PWR08"
+			(at 210.82 35.56 0)
+			(effects
+				(font
+					(size 1.27 1.27)
+				)
+				(hide yes)
+			)
+		)
+		(property "Value" "+5V"
+			(at 210.82 26.67 0)
+			(effects
+				(font
+					(size 1.27 1.27)
+				)
+			)
+		)
+		(property "Footprint" ""
+			(at 210.82 31.75 0)
+			(effects
+				(font
+					(size 1.27 1.27)
+				)
+				(hide yes)
+			)
+		)
+		(property "Datasheet" ""
+			(at 210.82 31.75 0)
+			(effects
+				(font
+					(size 1.27 1.27)
+				)
+				(hide yes)
+			)
+		)
+		(property "Description" "Power symbol creates a global label with name \"+5V\""
+			(at 210.82 31.75 0)
+			(effects
+				(font
+					(size 1.27 1.27)
+				)
+				(hide yes)
+			)
+		)
+		(pin "1"
+		)
+		(instances
+			(project ""
+				(path "/a7994af5-dcde-4bdd-b1f8-71f10278f6e4"
+					(reference "#PWR08")
+					(unit 1)
+				)
