File: telegram control.kicad_sch (KiCad schematic)
At the start: 13 parts, among them J1 Screw_Terminal_01x03, J2 Screw_Terminal_01x02, K1 SANYOU_SRD_Form_C, Q1 MMBT3904, U1 ESP32-C3_SUPERMINI_TH, U3 L7805

Commit message: telegram_control
Parts:
- removed J1: Screw_Terminal_01x03, TerminalBlock_Phoenix:TerminalBlock_Phoenix_MKDS-1,5-3_1x03_P5.00mm_Horizontal, symbol Connector:Screw_Terminal_01x03
- added J3: Conn_01x03_Pin, Connector_PinHeader_2.54mm:PinHeader_1x03_P2.54mm_Vertical, symbol Connector:Conn_01x03_Pin
- added J4: Screw_Terminal_01x02, TerminalBlock_Phoenix:TerminalBlock_Phoenix_MKDS-1,5-2_1x02_P5.00mm_Horizontal, symbol Connector:Screw_Terminal_01x02
Connections:
- net +5V: now also J3.3 (Pin_3)
- net GND: now also J3.1 (Pin_1)
- net gpio21: now reaches U1.21 (GPIO21)
- net gpio21: now also J3.2 (Pin_2)
- net at K1.1: now also J4.2 (Pin_2)
- net at K1.3: now also J4.1 (Pin_1)
