File: _autosave-telegram control.kicad_sch (KiCad schematic)
At the start: 13 parts, among them J1 Screw_Terminal_01x03, J2 Screw_Terminal_01x02, K1 SANYOU_SRD_Form_C, Q1 MMBT3904, U1 ESP32-C3_SUPERMINI_TH, U3 L7805

Commit message: telegram_control
Connections:
- net at R2.2: now also U1.0 (GPIO0); no longer U1.1 (GPIO1)
- net gpio0 renamed gpio1
- net gpio1: now also U1.1 (GPIO1); no longer U1.0 (GPIO0)
Other:
- moved on the sheet: D2, R2
Changed lines of the file:
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@@
+	(wire
+		(pts
+			(xy 123.19 67.31) (xy 127 67.31)
+		)
+		(stroke
+			(width 0)
+			(type default)
+		)
+	)
 	(wire
 		(pts
@@
 		)
 	)
-	(global_label "gpio0"
+	(global_label "gpio1"
 		(shape input)
-		(at 134.62 67.31 180)
+		(at 134.62 69.85 180)
 		(fields_autoplaced yes)
 		(effects
@@
 		)
 		(property "Intersheetrefs" "${INTERSHEET_REFS}"
-			(at 126.3735 67.31 0)
+			(at 126.3735 69.85 0)
 			(effects
 				(font
@@
 		)
 	)
-	(global_label "gpio0"
+	(global_label "gpio1"
 		(shape input)
 		(at 217.17 80.01 180)
@@
 	(symbol
 		(lib_id "Device:R")
-		(at 130.81 69.85 90)
+		(at 130.81 67.31 90)
 		(unit 1)
 		(exclude_from_sim no)
@@
 		(fields_autoplaced yes)
 		(property "Reference" "R2"
+			(at 130.81 60.96 90)
+			(effects
+				(font
+					(size 1.27 1.27)
+				)
+			)
+		)
+		(property "Value" "R"
 			(at 130.81 63.5 90)
 			(effects
@@
 			)
 		)
-		(property "Value" "R"
-			(at 130.81 66.04 90)
-			(effects
-				(font
-					(size 1.27 1.27)
-				)
-			)
-		)
 		(property "Footprint" "Resistor_SMD:R_1206_3216Metric"
-			(at 130.81 71.628 90)
+			(at 130.81 69.088 90)
 			(effects
 				(font
@@
 		)
 		(property "Datasheet" "~"
-			(at 130.81 69.85 0)
+			(at 130.81 67.31 0)
 			(effects
 				(font
@@
 		)
 		(property "Description" "Resistor"
-			(at 130.81 69.85 0)
+			(at 130.81 67.31 0)
 			(effects
 				(font
@@
 	(symbol
 		(lib_id "power:GND")
-		(at 127 77.47 0)
+		(at 123.19 74.93 0)
 		(unit 1)
 		(exclude_from_sim no)
@@
 		(fields_autoplaced yes)
 		(property "Reference" "#PWR03"
-			(at 127 83.82 0)
+			(at 123.19 81.28 0)
 			(effects
 				(font
@@
 		)
 		(property "Value" "GND"
-			(at 127 82.55 0)
+			(at 123.19 80.01 0)
 			(effects
 				(font
@@
 		)
 		(property "Footprint" ""
-			(at 127 77.47 0)
+			(at 123.19 74.93 0)
 			(effects
 				(font
@@
 		)
 		(property "Datasheet" ""
-			(at 127 77.47 0)
+			(at 123.19 74.93 0)
 			(effects
 				(font
@@
 		)
 		(property "Description" "Power symbol creates a global label with name \"GND\" , ground"
-			(at 127 77.47 0)
+			(at 123.19 74.93 0)
 			(effects
 				(font
@@
 	(symbol
 		(lib_id "Device:LED")
-		(at 127 73.66 90)
+		(at 123.19 71.12 90)
 		(unit 1)
 		(exclude_from_sim no)
@@
 		(fields_autoplaced yes)
 		(property "Reference" "D2"
-			(at 130.81 73.9774 90)
+			(at 127 71.4374 90)
 			(effects
 				(font
@@
 		)
 		(property "Value" "LED"
-			(at 130.81 76.5174 90)
+			(at 127 73.9774 90)
 			(effects
 				(font
@@
 		)
 		(property "Footprint" "LED_THT:LED_D3.0mm"
-			(at 127 73.66 0)
+			(at 123.19 71.12 0)
 			(effects
 				(font
@@
 		)
 		(property "Datasheet" "~"
-			(at 127 73.66 0)
+			(at 123.19 71.12 0)
 			(effects
 				(font
@@
 		)
 		(property "Description" "Light emitting diode"
-			(at 127 73.66 0)
+			(at 123.19 71.12 0)
 			(effects
 				(font
@@
 		)
 		(property "Sim.Pins" "1=K 2=A"
-			(at 127 73.66 0)
-			(effects
-				(font
+			(at 123.19 71.12 0)
+			(effects
+				(font
