File: telegram control.kicad_pcb (KiCad board)
At the start: 2 copper layers, 85.5 x 56 mm, 13 parts, among them J1 Screw_Terminal_01x03, J2 Screw_Terminal_01x02, K1 SANYOU_SRD_Form_C, Q1 MMBT3904, U1 ESP32-C3_SUPERMINI_TH, U3 L7805

Commit message: telegram_control
Parts:
- added G***: LOGO, logo:logo_1, F.Cu at (164.0, 98.0)
- added G***: LOGO, logo:logo_3, B.Cu at (198.0, 89.0)
- moved PS1 0.10 mm to (174.0, 82.6)

Commit message: telegram_control
Parts:
- removed the G*** at (198.0, 89.0)
- added G***: LOGO, logo:logo_2, B.Cu at (188.0, 84.5)
- PS1: footprint Converter_ACDC:Converter_ACDC_Hi-Link_HLK-10Mxx -> Converter_ACDC:Converter_ACDC_Hi-Link_HLK-PMxx
- moved U1 26.5 mm to (219.9, 86.9), turned to 0 degrees
- moved J2 1.50 mm to (163.3, 82.5)
Connections:
- C2 pad 1: Net-(U3-OUT) -> +5V
- R2 pad 2: Net-(U1-GPIO1) -> Net-(U1-GPIO0)
- R3 pad 1: gpio0 -> gpio1
- U1 pad 0: gpio0 -> Net-(U1-GPIO0)
- U1 pad 1: Net-(U1-GPIO1) -> gpio1
- U3 pad 3: Net-(U3-OUT) -> +5V
Routing:
- net +5V: track 0.00 -> 60.5 mm
- net Net-(U1-GPIO0): track 0.00 -> 34.3 mm, vias 0 -> 1
- net gpio1: track 0.00 -> 32.4 mm, vias 0 -> 1
- net Net-(U1-GPIO1): track 18.2 -> 0.00 mm
- net gpio0: track 16.6 -> 0.00 mm
- net Net-(U3-OUT): track 14.6 -> 0.00 mm
- net +12V: track 45.3 -> 42.6 mm, vias 1 -> 0
- net Net-(J2-Pin_2): track 11.3 -> 10.7 mm
- net Net-(J2-Pin_1): track 11.3 -> 10.7 mm
Other:
- board size 85.5 x 56 mm -> 75 x 53 mm

Commit message: telegram_control
Parts:
- moved G*** 2.06 mm to (166.0, 98.5)
Changed lines of the file:
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@@
 	(footprint "logo:logo_1"
 		(layer "F.Cu")
-		(at 164 98)
+		(at 166 98.5)
 		(property "Reference" "G***"
 			(at 5 -6.5 0)
@@
 		(layer "Edge.Cuts")
 	)
+	(dimension
+		(type aligned)
+		(layer "Edge.Cuts")
+		(pts
+			(xy 155 72) (xy 155 125)
+		)
+		(height 0)
+		(format
+			(prefix "")
+			(suffix "")
+			(units 3)
+			(units_format 0)
+			(precision 4)
+			(suppress_zeroes yes)
+		)
+		(style
+			(thickness 0.05)
+			(arrow_length 1.27)
+			(text_position_mode 0)
+			(arrow_direction outward)
+			(extension_height 0.58642)
+			(extension_offset 0.5)
+			(keep_text_aligned yes)
+		)
+		(gr_text "53"
+			(at 153.85 98.5 90)
+			(layer "Edge.Cuts")
+			(effects
+				(font
+					(size 1 1)
+					(thickness 0.15)
+				)
+			)
+		)
+	)
+	(dimension
+		(type aligned)
+		(layer "Edge.Cuts")
+		(pts
+			(xy 155 72) (xy 230 72)
+		)
+		(height 0)
+		(format
+			(prefix "")
+			(suffix "")
+			(units 3)
+			(units_format 0)
+			(precision 4)
+			(suppress_zeroes yes)
+		)
+		(style
+			(thickness 0.05)
+			(arrow_length 1.27)
+			(text_position_mode 0)
+			(arrow_direction outward)
+			(extension_height 0.58642)
+			(extension_offset 0.5)
+			(keep_text_aligned yes)
+		)
+		(gr_text "75"
+			(at 192.5 70.85 0)
+			(layer "Edge.Cuts")
+			(effects
+				(font
+					(size 1 1)
+					(thickness 0.15)
+				)
+			)
+		)
+	)
 	(segment

Commit message: telegram_control
Parts:
- removed J1: Screw_Terminal_01x03, TerminalBlock_Phoenix:TerminalBlock_Phoenix_MKDS-1,5-3_1x03_P5.00mm_Horizontal
- added J3: Conn_01x03_Pin, Connector_PinHeader_2.54mm:PinHeader_1x03_P2.54mm_Vertical, B.Cu at (192.5, 98.5)
- added J4: Screw_Terminal_01x02, TerminalBlock_Phoenix:TerminalBlock_Phoenix_MKDS-1,5-2_1x02_P5.00mm_Horizontal, F.Cu at (163.0, 107.5)
- moved G*** 15.7 mm to (180.0, 98.0)
- moved C1 7.50 mm to (204.5, 110.0), turned to 180 degrees
- moved C2 6.50 mm to (197.0, 110.0), turned to 0 degrees
- moved G*** 1.41 mm to (165.0, 99.5)
Connections:
- K1 pad 4: Net-(J1-Pin_3) -> unconnected-(K1-Pad4)
- U1 pad 21: unconnected-(U1-GPIO21-Pad21) -> gpio21
Routing:
- net gpio21: track 0.00 -> 22.4 mm
- net Net-(J1-Pin_3): track 11.8 -> 0.00 mm
- net +5V: track 60.5 -> 68.2 mm
- net +12V: track 42.6 -> 43.2 mm, vias 0 -> 2

Commit message: control por telegram
Parts:
- D2: moved to B.Cu
- moved D2 2.66 mm to (205.5, 120.0)
Other:
- outline, holes or cut-outs redrawn
- board text added: "Fase"
- board text added: "Lampara"
- board text added: "Neutro"

Commit message: control por telegram
Parts:
- moved D2 0.54 mm to (205.5, 119.5)
Changed lines of the file:
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@@
 	(footprint "LED_THT:LED_D3.0mm"
 		(layer "B.Cu")
-		(at 205.5 120.04 90)
+		(at 205.5 119.5 90)
 		(descr "LED, diameter 3.0mm, 2 pins, generated by kicad-footprint-generator")
 		(tags "LED")
@@
 		)
 	)
-	(dimension
-		(type orthogonal)
-		(layer "F.SilkS")
-		(pts
-			(xy 155 72) (xy 230 72)
-		)
-		(height 0)
-		(orientation 0)
-		(format
-			(prefix "")
-			(suffix "")
-			(units 3)
-			(units_format 0)
-			(precision 4)
-			(suppress_zeroes yes)
-		)
-		(style
-			(thickness 0.1)
-			(arrow_length 1.27)
-			(text_position_mode 0)
-			(arrow_direction outward)
-			(extension_height 0.58642)
-			(extension_offset 0.5)
-			(keep_text_aligned yes)
-		)
-		(gr_text "75"
-			(at 192.5 70.9 0)
-			(layer "F.SilkS")
-			(effects
-				(font
-					(size 1 1)
-					(thickness 0.1)
-				)
-			)
-		)
-	)
-	(dimension
-		(type orthogonal)
-		(layer "F.SilkS")
-		(pts
-			(xy 155 72) (xy 155 125)
-		)
-		(height 0)
-		(orientation 1)
-		(format
-			(prefix "")
-			(suffix "")
-			(units 3)
-			(units_format 0)
-			(precision 4)
-			(suppress_zeroes yes)
-		)
-		(style
-			(thickness 0.1)
-			(arrow_length 1.27)
-			(text_position_mode 0)
-			(arrow_direction outward)
-			(extension_height 0.58642)
-			(extension_offset 0.5)
-			(keep_text_aligned yes)
-		)
-		(gr_text "53"
-			(at 153.9 98.5 90)
-			(layer "F.SilkS")
-			(effects
-				(font
-					(size 1 1)
-					(thickness 0.1)
-				)
-			)
-		)
-	)
 	(segment
 		(start 197.5 97)
@@
 	)
 	(segment
-		(start 205.5 117.5)
-		(end 206 117.5)
+		(start 206 117.5)
+		(end 206 117.46)
 		(width 0.5)
 		(layer "F.Cu")
@@
 		(width 0.5)
 		(layer "F.Cu")
+		(net 16)
+	)
+	(segment
+		(start 206 117.46)
+		(end 205.5 116.96)
+		(width 0.5)
+		(layer "F.Cu")
